File: hw/power.sch (KiCad schematic (older format))
At the start: 8 parts, among them J4 4.5V Power Supply

Commit message: multiple changes
Parts:
- D1: value D_Small -> SS34; footprint (none) -> Diode_SMD:D_SMA
Changed lines of the file:
@@
 	2350 1850 2100 1850
-$Comp
-L Device:Jumper_NC_Small JP4
-U 1 1 5DC9629B
-P 4300 1750
-F 0 "JP4" H 4300 1962 50  0000 C CNN
-F 1 "5VA Bridge" H 4300 1871 50  0000 C CNN
-F 2 "Jumper:SolderJumper-2_P1.3mm_Bridged_RoundedPad1.0x1.5mm" H 4300 1750 50  0001 C CNN
-F 3 "~" H 4300 1750 50  0001 C CNN
-	1    4300 1750
-	1    0    0    -1
-$EndComp
 $Comp
 L power:+5VA #PWR0202
@@
 	1    0    0    -1
 $EndComp
-Wire Wire Line
-	4850 1600 4850 1750
-Wire Wire Line
-	4850 1750 4400 1750
-Wire Wire Line
-	4200 1750 3750 1750
 Connection ~ 3750 1750
 $Comp
@@
 	4000 2050 3750 2050
 Wire Wire Line
-	4500 2050 4200 2050
-Wire Wire Line
 	3750 2050 3750 1750
 Connection ~ 3750 2050
-Wire Wire Line
-	4850 1750 4850 2050
-Connection ~ 4850 1750
 Connection ~ 4850 2050
 $Comp
@@
 P 3450 1750
 F 0 "D1" H 3450 1545 50  0000 C CNN
-F 1 "D_Small" H 3450 1636 50  0000 C CNN
-F 2 "" V 3450 1750 50  0001 C CNN
+F 1 "SS34" H 3450 1636 50  0000 C CNN
+F 2 "Diode_SMD:D_SMA" V 3450 1750 50  0001 C CNN
 F 3 "~" V 3450 1750 50  0001 C CNN
 	1    3450 1750
 	-1   0    0    1
 $EndComp
+Wire Wire Line
+	4500 2050 4200 2050
+Wire Wire Line
+	4850 1750 4850 2050
+Wire Wire Line
+	4850 1600 4850 1750
+Connection ~ 4850 1750
+Wire Wire Line
+	4850 1750 4400 1750
+Wire Wire Line
+	4200 1750 3750 1750
+$Comp
+L Device:Jumper_NC_Small JP4
+U 1 1 5DC9629B
+P 4300 1750
+F 0 "JP4" H 4300 1962 50  0000 C CNN
+F 1 "5VA Bridge" H 4300 1871 50  0000 C CNN
+F 2 "Jumper:SolderJumper-2_P1.3mm_Bridged_RoundedPad1.0x1.5mm" H 4300 1750 50  0001 C CNN
+F 3 "~" H 4300 1750 50  0001 C CNN
+	1    4300 1750
+	1    0    0    -1
+$EndComp
 $EndSCHEMATC

Commit message: fix mux enable pin, reroute some traces
Parts:
- R68: value 4 -> 22
Connections:
- net +5VA: no longer JP4.2
- net at L1.1, R68.2: now also JP4.2
Changed lines of the file:
@@
 EESchema Schematic File Version 4
-LIBS:charger2-cache
 EELAYER 30 0
 EELAYER END
@@
 P 4600 2050
 F 0 "R68" V 4404 2050 50  0000 C CNN
-F 1 "4" V 4495 2050 50  0000 C CNN
+F 1 "22" V 4495 2050 50  0000 C CNN
 F 2 "Resistor_SMD:R_0805_2012Metric_Pad1.15x1.40mm_HandSolder" H 4600 2050 50  0001 C CNN
 F 3 "~" H 4600 2050 50  0001 C CNN
@@
 $EndComp
 Wire Wire Line
-	4500 2050 4200 2050
-Wire Wire Line
-	4850 1750 4850 2050
-Wire Wire Line
-	4850 1600 4850 1750
-Connection ~ 4850 1750
-Wire Wire Line
-	4850 1750 4400 1750
+	4500 2050 4400 2050
 Wire Wire Line
 	4200 1750 3750 1750
@@
 	1    0    0    -1
 $EndComp
+Wire Wire Line
+	4850 1600 4850 2050
+Wire Wire Line
+	4400 1750 4400 2050
+Connection ~ 4400 2050
+Wire Wire Line
+	4400 2050 4200 2050
 $EndSCHEMATC
