File: hw/power.sch (KiCad schematic (older format))
At the start: 8 parts, among them J4 4.5V Power Supply

Commit message: additional caps, groundplane improvements, MISO 3.3->5V
Connections:
- net VCC renamed VDD
Changed lines of the file:
@@
-$EndComp
-$Comp
-L power:VCC #PWR0199
-U 1 1 5DC935B5
-P 3100 1600
-F 0 "#PWR0199" H 3100 1450 50  0001 C CNN
-F 1 "VCC" H 3117 1773 50  0000 C CNN
-F 2 "" H 3100 1600 50  0001 C CNN
-F 3 "" H 3100 1600 50  0001 C CNN
-	1    3100 1600
-	1    0    0    -1
 $EndComp
 $Comp
@@
 Wire Wire Line
 	2500 1750 2100 1750
+$Comp
+L power:VDD #PWR?
+U 1 1 5FEBB3D5
+P 3100 1600
+F 0 "#PWR?" H 3100 1450 50  0001 C CNN
+F 1 "VDD" H 3115 1773 50  0000 C CNN
+F 2 "" H 3100 1600 50  0001 C CNN
+F 3 "" H 3100 1600 50  0001 C CNN
+	1    3100 1600
+	1    0    0    -1
+$EndComp
 $EndSCHEMATC
