File: hw/charger2.sch (KiCad schematic (older format))
At the start: 7 parts, among them J6 Temp, J7 Temp

Commit message: hw: pcb redesign
Parts:
- removed H3, H4: MountingHole, MountingHole:MountingHole_3.2mm_M3_ISO14580_Pad, symbol Mechanical:MountingHole
- removed J6, J7: Temp, Connector_PinHeader_2.54mm:PinHeader_1x03_P2.54mm_Vertical, symbol Connector_Generic:Conn_01x03
- removed R2: 4k7, Resistor_SMD:R_0805_2012Metric_Pad1.15x1.40mm_HandSolder, symbol Device:R_Small
Connections:
- no-connect marks 0 -> 3
Other:
- moved on the sheet: H1, H2
