File: hw/mcu.sch (KiCad schematic (older format))
At the start: 5 parts, among them SW1 Rotary_Encoder_Switch

Commit message: multiple changes
Parts:
- XA1: symbol charger2-rescue:Arduino_Nano_Socket-Arduino -> charger2-rescue:Arduino_Nano_Socket-Arduino-charger2-rescue
Changed lines of the file:
@@
 $Descr A4 11693 8268
 encoding utf-8
-Sheet 14 15
+Sheet 15 15
 Title ""
 Date ""
@@
 	3150 3750 3550 3750
 $Comp
-L charger2-rescue:Arduino_Nano_Socket-Arduino XA1
+L charger2-rescue:Arduino_Nano_Socket-Arduino-charger2-rescue XA1
 U 1 1 5DFF8FDC
 P 4850 4050

Commit message: hw: pcb redesign
Parts:
- SW1: value Rotary_Encoder_Switch -> Button
- XA1: value Arduino_Nano_Socket -> Arduino Nano
Connections:
- net D3 renamed FAN_PWM
- net D6 renamed TempS_A
- net D7 renamed TempS_B
Changed lines of the file:
@@
 EESchema Schematic File Version 4
-LIBS:charger2-cache
 EELAYER 30 0
 EELAYER END
 $Descr A4 11693 8268
 encoding utf-8
-Sheet 15 15
+Sheet 17 17
 Title ""
 Date ""
@@
 P 9500 3900
 F 0 "SW1" H 9500 4267 50  0000 C CNN
-F 1 "Rotary_Encoder_Switch" H 9500 4176 50  0000 C CNN
+F 1 "Button" H 9500 4176 50  0000 C CNN
 F 2 "Rotary_Encoder:RotaryEncoder_Alps_EC11E-Switch_Vertical_H20mm" H 9350 4060 50  0001 C CNN
 F 3 "~" H 9500 4160 50  0001 C CNN
@@
 NoConn ~ 3550 4350
 Text HLabel 6200 3650 2    50   Output ~ 0
-D7
+TempS_B
 Wire Wire Line
 	6200 3650 6150 3650
 Text HLabel 6200 3550 2    50   Output ~ 0
-D6
+TempS_A
 Wire Wire Line
 	6200 3550 6150 3550
@@
 A1
 Text HLabel 6150 3250 2    50   Output ~ 0
-D3
+FAN_PWM
 NoConn ~ 3550 4950
 Wire Wire Line
@@
 AR Path="/5DC57FBE/5DFF8FDC" Ref="XA1"  Part="1"
 F 0 "XA1" H 4850 5287 60  0000 C CNN
-F 1 "Arduino_Nano_Socket" H 4850 5181 60  0000 C CNN
+F 1 "Arduino Nano" H 4850 5181 60  0000 C CNN
 F 2 "arduino:Arduino_Nano_Socket" H 6650 7800 60  0001 C CNN
 F 3 "https://store.arduino.cc/arduino-nano" H 6650 7800 60  0001 C CNN
