File: hw/temp.sch (KiCad schematic (older format))
At the start: 1 part, among them U4 74HC4052

Commit message: fix 4052 footprint
Parts:
- U4: footprint Package_SO:SO-16_5.3x10.2mm_P1.27mm -> Package_SO:SO-16_3.9x9.9mm_P1.27mm
Changed lines of the file:
@@
 F 0 "U4" H 4150 4000 50  0000 C CNN
 F 1 "74HC4052" H 4100 3900 50  0000 C CNN
-F 2 "Package_SO:SO-16_5.3x10.2mm_P1.27mm" H 4300 3100 50  0001 C CNN
+F 2 "Package_SO:SO-16_3.9x9.9mm_P1.27mm" H 4300 3100 50  0001 C CNN
 F 3 "http://www.intersil.com/content/dam/Intersil/documents/cd40/cd4051bms-52bms-53bms.pdf" H 4300 3100 50  0001 C CNN
 	1    4300 3100
