File: hw/Battery.sch (KiCad schematic (older format))
At the start: 12 parts, among them Q1 AO3400, Q2 AO3400, U2 TP4056

Commit message: hw: pcb redesign
Parts:
- added R11: 47k, Resistor_SMD:R_0805_2012Metric_Pad1.20x1.40mm_HandSolder, symbol Device:R
- added R12: 3.6R, Resistor_THT:R_Axial_Power_L38.0mm_W9.0mm_P45.72mm, symbol Device:Heater
- added TH8: NTCLE100E3473, Resistor_THT:R_Axial_DIN0204_L3.6mm_D1.6mm_P1.90mm_Vertical, symbol Device:Thermistor_NTC
- BT1: footprint Connector_PinSocket_2.54mm:PinSocket_1x02_P2.54mm_Vertical -> Battery:BatteryHolder_MPD_BH-18650-PC2
- U2: footprint Package_SO:SOP-8-1EP_4.57x4.57mm_P1.27mm_EP4.57x4.45mm_ThermalVias -> TP4056:TP4056_SOP-8-PP
Connections:
- net Bat+: no longer Q2.1 (G)
- net GND: now also TH8.2
- net L+ renamed Bat+'
- net Bat+': now also Q2.1 (G), R12.1
- net L-: no longer names the net of Q1.3 (D)
- net L-: now also R12.2
- new net +5VA: R11.1
- new net TEMP: R11.2, TH8.1
Other:
- moved on the sheet: R32, R33

Commit message: additional caps, groundplane improvements, MISO 3.3->5V
Connections:
- net VCC renamed VDD
Changed lines of the file:
@@
 $Descr A4 11693 8268
 encoding utf-8
-Sheet 3 17
+Sheet 5 17
 Title ""
 Date ""
@@
 AR Path="/5DE37049/5DC5D9F3/5DD277B3" Ref="#PWR?"  Part="1"
 AR Path="/5DE37049/5DC5DB65/5DD277B3" Ref="#PWR?"  Part="1"
-F 0 "#PWR0143" H 5100 3000 50  0001 C CNN
+F 0 "#PWR0122" H 5100 3000 50  0001 C CNN
 F 1 "GND" H 5105 3077 50  0000 C CNN
 F 2 "" H 5100 3250 50  0001 C CNN
@@
 AR Path="/5DE37049/5DC5D9F3/5DBBD668" Ref="#PWR?"  Part="1"
 AR Path="/5DE37049/5DC5DB65/5DBBD668" Ref="#PWR?"  Part="1"
-F 0 "#PWR0144" H 6200 3100 50  0001 C CNN
+F 0 "#PWR0123" H 6200 3100 50  0001 C CNN
 F 1 "GND" H 6205 3177 50  0000 C CNN
 F 2 "" H 6200 3350 50  0001 C CNN
@@
 Wire Wire Line
 	6200 3150 6200 3350
-$Comp
-L power:VCC #PWR0111
-U 1 1 5DC3D6EE
-P 3150 2400
-AR Path="/5DBBB1EF/5DC3D6EE" Ref="#PWR0111"  Part="1"
-AR Path="/5DC54FE6/5DC3D6EE" Ref="#PWR?"  Part="1"
-AR Path="/5DC563B3/5DC3D6EE" Ref="#PWR?"  Part="1"
-AR Path="/5DC58B11/5DC3D6EE" Ref="#PWR0118"  Part="1"
-AR Path="/5DC59791/5DC3D6EE" Ref="#PWR0125"  Part="1"
-AR Path="/5DC5994B/5DC3D6EE" Ref="#PWR0132"  Part="1"
-AR Path="/5DC5B1E5/5DC3D6EE" Ref="#PWR0139"  Part="1"
-AR Path="/5DC5B1EC/5DC3D6EE" Ref="#PWR0146"  Part="1"
-AR Path="/5DC5B1F3/5DC3D6EE" Ref="#PWR0153"  Part="1"
-AR Path="/5DC5B1FA/5DC3D6EE" Ref="#PWR0160"  Part="1"
-AR Path="/5E0C52EA/5DC3D6EE" Ref="#PWR0189"  Part="1"
-AR Path="/5E0C52F1/5DC3D6EE" Ref="#PWR0196"  Part="1"
-AR Path="/5E0C52F8/5DC3D6EE" Ref="#PWR0203"  Part="1"
-AR Path="/5E0C5314/5DC3D6EE" Ref="#PWR0210"  Part="1"
-AR Path="/5DC581CC/5DC581FA/5DC3D6EE" Ref="#PWR0124"  Part="1"
-AR Path="/5DC581CC/5DC5D939/5DC3D6EE" Ref="#PWR0131"  Part="1"
-AR Path="/5DC581CC/5DC5D9F3/5DC3D6EE" Ref="#PWR0138"  Part="1"
-AR Path="/5DC581CC/5DC5DB65/5DC3D6EE" Ref="#PWR0145"  Part="1"
-AR Path="/5DC82B0A/5DC581FA/5DC3D6EE" Ref="#PWR0166"  Part="1"
-AR Path="/5DC82B0A/5DC5D939/5DC3D6EE" Ref="#PWR0173"  Part="1"
-AR Path="/5DC82B0A/5DC5D9F3/5DC3D6EE" Ref="#PWR0180"  Part="1"
-AR Path="/5DC82B0A/5DC5DB65/5DC3D6EE" Ref="#PWR0187"  Part="1"
-AR Path="/5DE36E4E/5DC581FA/5DC3D6EE" Ref="#PWR?"  Part="1"
-AR Path="/5DE36E4E/5DC5D939/5DC3D6EE" Ref="#PWR?"  Part="1"
-AR Path="/5DE36E4E/5DC5D9F3/5DC3D6EE" Ref="#PWR?"  Part="1"
-AR Path="/5DE36E4E/5DC5DB65/5DC3D6EE" Ref="#PWR?"  Part="1"
-AR Path="/5DE37049/5DC581FA/5DC3D6EE" Ref="#PWR?"  Part="1"
-AR Path="/5DE37049/5DC5D939/5DC3D6EE" Ref="#PWR?"  Part="1"
-AR Path="/5DE37049/5DC5D9F3/5DC3D6EE" Ref="#PWR?"  Part="1"
-AR Path="/5DE37049/5DC5DB65/5DC3D6EE" Ref="#PWR?"  Part="1"
-F 0 "#PWR0145" H 3150 2250 50  0001 C CNN
-F 1 "VCC" H 3167 2573 50  0000 C CNN
-F 2 "" H 3150 2400 50  0001 C CNN
-F 3 "" H 3150 2400 50  0001 C CNN
-	1    3150 2400
-	1    0    0    -1
-$EndComp
 Wire Wire Line
 	3150 2400 3150 2450
@@
 AR Path="/5DE37049/5DC5D9F3/5DD277C5" Ref="#PWR?"  Part="1"
 AR Path="/5DE37049/5DC5DB65/5DD277C5" Ref="#PWR?"  Part="1"
-F 0 "#PWR0146" H 9400 3350 50  0001 C CNN
+F 0 "#PWR0125" H 9400 3350 50  0001 C CNN
 F 1 "GND" H 9405 3427 50  0000 C CNN
 F 2 "" H 9400 3600 50  0001 C CNN
@@
 AR Path="/5DE37049/5DC5D9F3/5DC5E196" Ref="#PWR?"  Part="1"
 AR Path="/5DE37049/5DC5DB65/5DC5E196" Ref="#PWR?"  Part="1"
-F 0 "#PWR0147" H 7950 3450 50  0001 C CNN
+F 0 "#PWR0126" H 7950 3450 50  0001 C CNN
 F 1 "GND" H 7955 3527 50  0000 C CNN
 F 2 "" H 7950 3700 50  0001 C CNN
@@
 AR Path="/5DE37049/5DC5D9F3/5DC7184E" Ref="R?"  Part="1"
 AR Path="/5DE37049/5DC5DB65/5DC7184E" Ref="R?"  Part="1"
-F 0 "R29" H 5759 3046 50  0000 L CNN
+F 0 "R5" H 5759 3046 50  0000 L CNN
 F 1 "1k2" H 5759 2955 50  0000 L CNN
 F 2 "Resistor_SMD:R_0805_2012Metric_Pad1.15x1.40mm_HandSolder" H 5700 3000 50  0001 C CNN
@@
 AR Path="/5DE37049/5DC5D9F3/5DD277B6" Ref="R?"  Part="1"
 AR Path="/5DE37049/5DC5DB65/5DD277B6" Ref="R?"  Part="1"
-F 0 "R30" H 7559 3546 50  0000 L CNN
+F 0 "R6" H 7559 3546 50  0000 L CNN
 F 1 "10k" H 7559 3455 50  0000 L CNN
 F 2 "Resistor_SMD:R_0805_2012Metric_Pad1.15x1.40mm_HandSolder" H 7500 3500 50  0001 C CNN
@@
 AR Path="/5DE37049/5DC5D9F3/5DD277B8" Ref="R?"  Part="1"
 AR Path="/5DE37049/5DC5DB65/5DD277B8" Ref="R?"  Part="1"
-F 0 "R34" H 9159 2146 50  0000 L CNN
+F 0 "R10" H 9159 2146 50  0000 L CNN
 F 1 "470" H 9159 2055 50  0000 L CNN
 F 2 "Resistor_SMD:R_0805_2012Metric_Pad1.15x1.40mm_HandSolder" H 9100 2100 50  0001 C CNN
@@
 AR Path="/5DE37049/5DC5D9F3/5DD277B9" Ref="C?"  Part="1"
 AR Path="/5DE37049/5DC5DB65/5DD277B9" Ref="C?"  Part="1"
-F 0 "C8" H 5992 2646 50  0000 L CNN
+F 0 "C2" H 5992 2646 50  0000 L CNN
 F 1 "10u" H 5992 2555 50  0000 L CNN
 F 2 "Capacitor_SMD:C_0805_2012Metric_Pad1.15x1.40mm_HandSolder" H 5900 2600 50  0001 C CNN
@@
 AR Path="/5DE37049/5DC5D9F3/5DD277BB" Ref="#PWR?"  Part="1"
 AR Path="/5DE37049/5DC5DB65/5DD277BB" Ref="#PWR?"  Part="1"
-F 0 "#PWR0148" H 3200 2600 50  0001 C CNN
+F 0 "#PWR0127" H 3200 2600 50  0001 C CNN
 F 1 "GND" H 3205 2677 50  0000 C CNN
 F 2 "" H 3200 2850 50  0001 C CNN
@@
 AR Path="/5DE37049/5DC5D9F3/5DD277BA" Ref="C?"  Part="1"
 AR Path="/5DE37049/5DC5DB65/5DD277BA" Ref="C?"  Part="1"
-F 0 "C7" H 3292 2696 50  0000 L CNN
+F 0 "C1" H 3292 2696 50  0000 L CNN
 F 1 "10u" H 3292 2605 50  0000 L CNN
 F 2 "Capacitor_SMD:C_0805_2012Metric_Pad1.15x1.40mm_HandSolder" H 3200 2650 50  0001 C CNN
@@
 AR Path="/5DE37049/5DC5D9F3/5DC4807B" Ref="R?"  Part="1"
 AR Path="/5DE37049/5DC5DB65/5DC4807B" Ref="R?"  Part="1"
-F 0 "R33" H 9009 2696 50  0000 L CNN
+F 0 "R9" H 9009 2696 50  0000 L CNN
 F 1 "10k" H 9009 2605 50  0000 L CNN
 F 2 "Resistor_SMD:R_0805_2012Metric_Pad1.15x1.40mm_HandSolder" H 8950 2650 50  0001 C CNN
@@
 AR Path="/5DE37049/5DC5D9F3/5DD277C1" Ref="BT?"  Part="1"
 AR Path="/5DE37049/5DC5DB65/5DD277C1" Ref="BT?"  Part="1"
-F 0 "BT4" H 9518 2996 50  0000 L CNN
+F 0 "BT1" H 9518 2996 50  0000 L CNN
 F 1 "Battery_Cell" H 9518 2905 50  0000 L CNN
 F 2 "Battery:BatteryHolder_MPD_BH-18650-PC2" V 9400 2960 50  0001 C CNN
@@
 AR Path="/5DE37049/5DC5D9F3/5DC270F2" Ref="R?"  Part="1"
 AR Path="/5DE37049/5DC5DB65/5DC270F2" Ref="R?"  Part="1"
-F 0 "R31" V 8154 2200 50  0000 C CNN
+F 0 "R7" V 8154 2200 50  0000 C CNN
 F 1 "470" V 8245 2200 50  0000 C CNN
 F 2 "Resistor_SMD:R_0805_2012Metric_Pad1.15x1.40mm_HandSolder" H 8350 2200 50  0001 C CNN
@@
 AR Path="/5DE37049/5DC5D9F3/5E1D2F9B" Ref="R?"  Part="1"
 AR Path="/5DE37049/5DC5DB65/5E1D2F9B" Ref="R?"  Part="1"
-F 0 "R32" H 8759 2496 50  0000 L CNN
+F 0 "R8" H 8759 2496 50  0000 L CNN
 F 1 "20m" H 8759 2405 50  0000 L CNN
 F 2 "Resistor_SMD:R_1206_3216Metric_Pad1.42x1.75mm_HandSolder" H 8700 2450 50  0001 C CNN
@@
 AR Path="/5DE37049/5DC5D9F3/5DD277B2" Ref="U?"  Part="1"
 AR Path="/5DE37049/5DC5DB65/5DD277B2" Ref="U?"  Part="1"
-F 0 "U10" H 5100 3237 60  0000 C CNN
+F 0 "U7" H 5100 3237 60  0000 C CNN
 F 1 "TP4056" H 5100 3131 60  0000 C CNN
 F 2 "TP4056:TP4056_SOP-8-PP" H 5100 2700 60  0001 C CNN
@@
 AR Path="/5DE37049/5DC5D9F3/5DD277C3" Ref="Q?"  Part="1"
 AR Path="/5DE37049/5DC5DB65/5DD277C3" Ref="Q?"  Part="1"
-F 0 "Q9" H 9506 3246 50  0000 L CNN
+F 0 "Q3" H 9506 3246 50  0000 L CNN
 F 1 "AO3400" H 9506 3155 50  0000 L CNN
 F 2 "Package_TO_SOT_SMD:SOT-23_Handsoldering" H 9500 3300 50  0001 C CNN
@@
 AR Path="/5DE37049/5DC5D9F3/5DC209D5" Ref="Q?"  Part="1"
 AR Path="/5DE37049/5DC5DB65/5DC209D5" Ref="Q?"  Part="1"
-F 0 "Q8" H 8056 3446 50  0000 L CNN
+F 0 "Q2" H 8056 3446 50  0000 L CNN
 F 1 "AO3400" H 8056 3355 50  0000 L CNN
 F 2 "Package_TO_SOT_SMD:SOT-23_Handsoldering" H 8050 3500 50  0001 C CNN
@@
 AR Path="/5DC82B0A/5DC5D9F3/5F95C6DE" Ref="R36"  Part="1"
 AR Path="/5DC82B0A/5DC5DB65/5F95C6DE" Ref="R28"  Part="1"
-F 0 "R2" H 8020 2896 50  0000 L CNN
+F 0 "R12" H 8020 2896 50  0000 L CNN
 F 1 "3.6R" H 8020 2805 50  0000 L CNN
 F 2 "Resistor_THT:R_Axial_Power_L38.0mm_W9.0mm_P45.72mm" V 7880 2850 50  0001 C CNN
@@
 AR Path="/5DC82B0A/5DC5DB65/5F9AFDBE" Ref="TH5"  Part="1"
 AR Path="/5DC82B0A/5DC5D9F3/5F9AFDBE" Ref="TH6"  Part="1"
-F 0 "TH1" H 7148 5496 50  0000 L CNN
+F 0 "TH3" H 7148 5496 50  0000 L CNN
 F 1 "NTCLE100E3473" H 7148 5405 50  0000 L CNN
 F 2 "Resistor_THT:R_Axial_DIN0204_L3.6mm_D1.6mm_P1.90mm_Vertical" H 7050 5500 50  0001 C CNN
@@
 AR Path="/5DC82B0A/5DC5DB65/5F9B247D" Ref="#PWR0163"  Part="1"
 AR Path="/5DC82B0A/5DC5D9F3/5F9B247D" Ref="#PWR0193"  Part="1"
-F 0 "#PWR0120" H 7050 4450 50  0001 C CNN
+F 0 "#PWR0157" H 7050 4450 50  0001 C CNN
 F 1 "+5VA" H 7065 4773 50  0000 C CNN
 F 2 "" H 7050 4600 50  0001 C CNN
@@
 AR Path="/5DC82B0A/5DC581FA/5F9B9C8B" Ref="#PWR0196"  Part="1"
 AR Path="/5DC82B0A/5DC5D939/5F9B9C8B" Ref="#PWR0198"  Part="1"
-F 0 "#PWR0121" H 7050 5550 50  0001 C CNN
+F 0 "#PWR0158" H 7050 5550 50  0001 C CNN
 F 1 "GND" H 7055 5627 50  0000 C CNN
 F 2 "" H 7050 5800 50  0001 C CNN
@@
 AR Path="/5DC82B0A/5DC581FA/5F9BEBD1" Ref="R37"  Part="1"
 AR Path="/5DC82B0A/5DC5D939/5F9BEBD1" Ref="R45"  Part="1"
-F 0 "R1" H 7120 4796 50  0000 L CNN
+F 0 "R11" H 7120 4796 50  0000 L CNN
 F 1 "47k" H 7120 4705 50  0000 L CNN
 F 2 "Resistor_SMD:R_0805_2012Metric_Pad1.20x1.40mm_HandSolder" V 6980 4750 50  0001 C CNN
@@
 AR Path="/5DE37049/5DC5D9F3/5DC4E17D" Ref="#PWR?"  Part="1"
 AR Path="/5DE37049/5DC5DB65/5DC4E17D" Ref="#PWR?"  Part="1"
-F 0 "#PWR0149" H 8950 2600 50  0001 C CNN
+F 0 "#PWR0128" H 8950 2600 50  0001 C CNN
 F 1 "GND" H 8955 2677 50  0000 C CNN
 F 2 "" H 8950 2850 50  0001 C CNN
@@
 Wire Wire Line
 	8950 2450 9100 2450
+$Comp
+L power:VDD #PWR?
+U 1 1 5FEBD477
+P 3150 2400
+F 0 "#PWR?" H 3150 2250 50  0001 C CNN
+F 1 "VDD" H 3165 2573 50  0000 C CNN
+F 2 "" H 3150 2400 50  0001 C CNN
+F 3 "" H 3150 2400 50  0001 C CNN
+	1    3150 2400
+	1    0    0    -1
+$EndComp
 $EndSCHEMATC
